File: DOCS/SCH-EAGLE/BLL-EBOOK.brd (EAGLE design)
At the start: 99.2 x 61.7 mm, 57 parts, among them IC1 RT9080-33GJ5, J1 541323462, J2 MSD-3-A, J3 DX07S016JA1R1500, Q1 IRLML6402TRPBF, U2 TPS65185RGZR, U3 USBLC6-2P6

Commit message: new pcb and sch files
Parts:
- removed JP1, JP2: (no value), pinhead:1X01
- added F1: 1206L150, SparkFun-Fuses:1206
- added J4: BATT PAD, pinhead:1X02/90
- added U$2: MINI360-MOD-REG, MINI360 MOD REGULATOR:MINI360
- moved C24 4.24 mm to (91.3, 73.2), turned to 0 degrees
- moved R12 2.69 mm to (94.8, 74.7), turned to 0 degrees
- moved L2 1.58 mm to (88.2, 70.9)
- moved C27 1.35 mm to (75.7, 48.7)
- moved R13 1.26 mm to (91.5, 74.8), turned to 0 degrees
- moved C20 1.26 mm to (87.1, 75.0), turned to 0 degrees
- moved C6 0.98 mm to (87.0, 73.1), turned to 180 degrees
- moved C5 0.77 mm to (72.9, 48.6)
- moved D10 0.71 mm to (90.4, 70.6)
- moved C28 0.56 mm to (71.1, 48.6)
- moved C25 0.48 mm to (92.0, 70.7)
Connections:
- removed net VCC: C27.A, C28.1, C5.1, JP1.1, U$1.79, U$1.80, U$1.81
- new net IN+: U$2.IN+
- new net OUT+: F1.2, U$2.OUT+
- new net P: C27.A, C28.1, C5.1, F1.1, U$1.79, U$1.80, U$1.81
- net GND: now also J4.2, U$2.IN-, U$2.OUT-; no longer JP2.1
- net VBAT: now also J4.1
Routing:
- net GND: track 493.9 -> 539.1 mm, vias 10 -> 11
- net VCC: track 21.3 -> 0.00 mm
- net VBAT: track 2.24 -> 23.2 mm, vias 0 -> 2
- net P: track 0.00 -> 13.1 mm
- net -15V: track 67.3 -> 80.0 mm
- net P37: track 12.6 -> 18.2 mm
- net +22V: track 110.9 -> 116.3 mm
- net VNEG-IN: track 17.9 -> 21.7 mm, vias 2 -> 3
- net OUT+: track 0.00 -> 3.75 mm
- net SDA: track 61.1 -> 64.4 mm
- net SCL: track 63.2 -> 66.2 mm
- net P40: track 3.71 -> 5.79 mm
- net P33: track 12.0 -> 13.7 mm
- net USB+: track 69.0 -> 70.1 mm
- net 15V: track 132.8 -> 131.8 mm
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Other:
- board text added: "- +"
- board text added: "IN FROM BAT"
- board text added: "to charge module"
