File: DOCS/SCH-EAGLE/BLL-EBOOK.sch (EAGLE design)
At the start: 57 parts, among them IC1 RT9080-33GJ5, J1 541323462, J2 MSD-3-A, J3 DX07S016JA1R1500, Q1 IRLML6402TRPBF, U2 TPS65185RGZR, U3 USBLC6-2P6

Commit message: new pcb and sch files
Parts:
- removed JP1, JP2: (no value), pinhead:PINHD-1X1
- added F1: 1206L150, SparkFun-Fuses:PPTC_6V500MA-2
- added J4: BATT PAD, pinhead:PINHD-1X2/90
- added U$2: MINI360-MOD-REG, MINI360 MOD REGULATOR:MINI360-MOD-REG
Connections:
- removed net VCC: C27.+, C28.1, C5.1, JP1.1, U$1.VCC5V1_SYS, U$1.VCC5V2_SYS, U$1.VCC5V3_SYS
- new net IN+: U$2.IN+
- new net OUT+: F1.2, U$2.OUT+
- new net P: C27.+, C28.1, C5.1, F1.1, U$1.VCC5V1_SYS, U$1.VCC5V2_SYS, U$1.VCC5V3_SYS
- net GND: now also J4.2, U$2.IN-, U$2.OUT-; no longer JP2.1
- net VBAT: now also J4.1
Other:
- note added: "SoM Power +5V-VCC"
Changed lines of the file:
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@@
 <part name="C27" library="SparkFun-Capacitors" deviceset="100UF-POLAR" device="-EIA3528-10V-20%(TANT)" value="100uF"/>
 <part name="C28" library="SparkFun-Capacitors" deviceset="CAP" device="-0805" value="100nF"/>
+<part name="U$2" library="MINI360 MOD REGULATOR" deviceset="MINI360-MOD-REG" device=""/>
 <part name="SUPPLY11" library="supply2" library_urn="urn:adsk.eagle:library:372" deviceset="GND" device=""/>
-<part name="JP1" library="pinhead" library_urn="urn:adsk.eagle:library:325" deviceset="PINHD-1X1" device="" package3d_urn="urn:adsk.eagle:package:22485/2"/>
-<part name="JP2" library="pinhead" library_urn="urn:adsk.eagle:library:325" deviceset="PINHD-1X1" device="" package3d_urn="urn:adsk.eagle:package:22485/2"/>
+<part name="SUPPLY12" library="supply2" library_urn="urn:adsk.eagle:library:372" deviceset="GND" device=""/>
+<part name="F1" library="SparkFun-Fuses" deviceset="PPTC" device="_6V500MA-2" value="1206L150"/>
+<part name="SUPPLY41" library="supply2" library_urn="urn:adsk.eagle:library:372" deviceset="GND" device=""/>
+<part name="J4" library="pinhead" library_urn="urn:adsk.eagle:library:325" deviceset="PINHD-1X2" device="/90" package3d_urn="urn:adsk.eagle:package:22437/2" value="BATT PAD"/>
+<part name="SUPPLY42" library="supply2" library_urn="urn:adsk.eagle:library:372" deviceset="GND" device=""/>
 </parts>
 <sheets>
@@
 <text x="-86.36" y="83.82" size="4.5" layer="91">PUERTO MICRO SD</text>
 <text x="-220.98" y="27.94" size="4.5" layer="91">PWR 3.3V</text>
-<text x="-137.16" y="22.86" size="4.5" layer="91">battery/usb
+<text x="-144.78" y="22.86" size="4.5" layer="91">battery/usb
 switching</text>
 <text x="-226.06" y="-20.32" size="4.5" layer="91">ePaper Display Power</text>
@@
 <text x="17.78" y="119.38" size="10.16" layer="94" font="vector" ratio="10" align="bottom-center">BLL Ebook Reader
 Based on Luckfox Core RV1106</text>
+<text x="-55.88" y="0" size="4.5" layer="91" rot="R90">SoM Power
++5V-VCC</text>
 </plain>
 <instances>
@@
 <attribute name="VALUE" x="141.859" y="24.384" size="1.778" layer="96" font="vector" rot="R90"/>
 </instance>
-<instance part="SUPPLY11" gate="GND" x="165.1" y="22.86" smashed="yes">
-<attribute name="VALUE" x="163.195" y="19.685" size="1.778" layer="96"/>
-</instance>
-<instance part="JP1" gate="G$1" x="167.64" y="40.64" smashed="yes" rot="R90">
-<attribute name="NAME" x="164.465" y="34.29" size="1.778" layer="95" rot="R90"/>
-<attribute name="VALUE" x="172.72" y="34.29" size="1.778" layer="96" rot="R90"/>
-</instance>
-<instance part="JP2" gate="G$1" x="172.72" y="25.4" smashed="yes">
-<attribute name="NAME" x="166.37" y="28.575" size="1.778" layer="95"/>
-<attribute name="VALUE" x="166.37" y="20.32" size="1.778" layer="96"/>
+<instance part="U$2" gate="G$2" x="-40.64" y="12.7" smashed="yes" rot="R90"/>
+<instance part="SUPPLY11" gate="GND" x="-81.28" y="-5.08" smashed="yes">
+<attribute name="VALUE" x="-83.185" y="-8.255" size="1.778" layer="96"/>
+</instance>
+<instance part="SUPPLY12" gate="GND" x="170.18" y="22.86" smashed="yes">
+<attribute name="VALUE" x="168.275" y="19.685" size="1.778" layer="96"/>
+</instance>
+<instance part="F1" gate="F1" x="167.64" y="43.18" smashed="yes" rot="R90">
+<attribute name="NAME" x="164.465" y="45.085" size="1.778" layer="95" font="vector" rot="R90" align="bottom-center"/>
+<attribute name="VALUE" x="170.434" y="44.45" size="1.778" layer="96" font="vector" rot="R90" align="top-center"/>
+</instance>
+<instance part="SUPPLY41" gate="GND" x="-7.62" y="-5.08" smashed="yes">
+<attribute name="VALUE" x="-9.525" y="-8.255" size="1.778" layer="96"/>
+</instance>
+<instance part="J4" gate="G$1" x="-93.98" y="20.32" smashed="yes">
+<attribute name="VALUE" x="-111.76" y="25.654" size="1.778" layer="96" font="vector"/>
+<attribute name="NAME" x="-96.52" y="25.908" size="1.778" layer="95" font="vector"/>
+</instance>
+<instance part="SUPPLY42" gate="GND" x="-104.14" y="17.78" smashed="yes">
+<attribute name="VALUE" x="-103.505" y="17.145" size="1.778" layer="96"/>
 </instance>
 </instances>
@@
 </segment>
 <segment>
+<pinref part="U$2" gate="G$2" pin="OUT-"/>
+<pinref part="SUPPLY11" gate="GND" pin="GND"/>
+<wire x1="-78.74" y1="-2.54" x2="-81.28" y2="-2.54" width="0.1524" layer="91"/>
+</segment>
+<segment>
 <pinref part="C28" gate="G$1" pin="2"/>
 <pinref part="C5" gate="G$1" pin="2"/>
@@
 <wire x1="154.94" y1="25.4" x2="149.86" y2="25.4" width="0.1524" layer="91"/>
 <junction x="149.86" y="25.4"/>
-<pinref part="SUPPLY11" gate="GND" pin="GND"/>
-<wire x1="154.94" y1="25.4" x2="165.1" y2="25.4" width="0.1524" layer="91"/>
+<wire x1="154.94" y1="25.4" x2="170.18" y2="25.4" width="0.1524" layer="91"/>
 <junction x="154.94" y="25.4"/>
-<pinref part="JP2" gate="G$1" pin="1"/>
-<wire x1="170.18" y1="25.4" x2="165.1" y2="25.4" width="0.1524" layer="91"/>
-<junction x="165.1" y="25.4"/>
+<label x="165.1" y="25.4" size="1.778" layer="95"/>
+<pinref part="SUPPLY12" gate="GND" pin="GND"/>
+</segment>
+<segment>
+<pinref part="U$2" gate="G$2" pin="IN-"/>
+<wire x1="-12.7" y1="-2.54" x2="-7.62" y2="-2.54" width="0.1524" layer="91"/>
+<label x="-10.16" y="-2.54" size="1.778" layer="95"/>
+<pinref part="SUPPLY41" gate="GND" pin="GND"/>
+</segment>
+<segment>
+<pinref part="J4" gate="G$1" pin="2"/>
+<pinref part="SUPPLY42" gate="GND" pin="GND"/>
+<wire x1="-104.14" y1="20.32" x2="-96.52" y2="20.32" width="0.1524" layer="91"/>
 </segment>
 </net>
@@
 <junction x="-134.62" y="12.7"/>
 </segment>
+<segment>
+<pinref part="J4" gate="G$1" pin="1"/>
+<wire x1="-96.52" y1="22.86" x2="-114.3" y2="22.86" width="0.1524" layer="91"/>
+<label x="-111.76" y="22.86" size="1.778" layer="95"/>
+</segment>
 </net>
 <net name="N$5" class="0">
@@
 </segment>
 </net>
-<net name="VCC" class="0">
-<segment>
-<pinref part="U$1" gate="G$1" pin="VCC5V3_SYS"/>
-<pinref part="U$1" gate="G$1" pin="VCC5V2_SYS"/>
-<wire x1="137.16" y1="35.56" x2="137.16" y2="33.02" width="0.1524" layer="91"/>
-<pinref part="U$1" gate="G$1" pin="VCC5V1_SYS"/>
-<wire x1="137.16" y1="30.48" x2="137.16" y2="33.02" width="0.1524" layer="91"/>
-<junction x="137.16" y="33.02"/>
-<wire x1="137.16" y1="33.02" x2="144.78" y2="33.02" width="0.1524" layer="91"/>
-<label x="149.86" y="35.56" size="1.778" layer="95" rot="R180"/>
-<pinref part="C27" gate="G$1" pin="+"/>
-<wire x1="144.78" y1="33.02" x2="149.86" y2="33.02" width="0.1524" layer="91"/>
-<wire x1="149.86" y1="33.02" x2="154.94" y2="33.02" width="0.1524" layer="91"/>
-<junction x="154.94" y="33.02"/>
-<pinref part="C28" gate="G$1" pin="1"/>
-<junction x="144.78" y="33.02"/>
-<pinref part="C5" gate="G$1" pin="1"/>
-<junction x="149.86" y="33.02"/>
-<wire x1="154.94" y1="33.02" x2="167.64" y2="33.02" width="0.1524" layer="91"/>
-<pinref part="JP1" gate="G$1" pin="1"/>
-<wire x1="167.64" y1="33.02" x2="167.64" y2="38.1" width="0.1524" layer="91"/>
+<net name="OUT+" class="0">
+<segment>
+<pinref part="U$2" gate="G$2" pin="OUT+"/>
+<wire x1="-78.74" y1="27.94" x2="-83.82" y2="27.94" width="0.1524" layer="91"/>
+<label x="-83.82" y="25.4" size="1.778" layer="95"/>
+</segment>
+<segment>
+<pinref part="F1" gate="F1" pin="2"/>
+<wire x1="167.64" y1="50.8" x2="167.64" y2="55.88" width="0.1524" layer="91"/>
+<label x="167.64" y="53.34" size="1.778" layer="95" rot="R90"/>
 </segment>
 </net>
@@
 </segment>
 </net>
+<net name="IN+" class="0">
+<segment>
+<pinref part="U$2" gate="G$2" pin="IN+"/>
+<wire x1="-12.7" y1="27.94" x2="-7.62" y2="27.94" width="0.1524" layer="91"/>
+<label x="-10.16" y="27.94" size="1.778" layer="95"/>
+</segment>
+</net>
+<net name="P" class="0">
+<segment>
+<pinref part="U$1" gate="G$1" pin="VCC5V3_SYS"/>
+<pinref part="U$1" gate="G$1" pin="VCC5V2_SYS"/>
+<wire x1="137.16" y1="35.56" x2="137.16" y2="33.02" width="0.1524" layer="91"/>
+<pinref part="U$1" gate="G$1" pin="VCC5V1_SYS"/>
+<wire x1="137.16" y1="30.48" x2="137.16" y2="33.02" width="0.1524" layer="91"/>
+<junction x="137.16" y="33.02"/>
+<wire x1="137.16" y1="33.02" x2="144.78" y2="33.02" width="0.1524" layer="91"/>
+<label x="165.1" y="35.56" size="1.778" layer="95" rot="R180"/>
+<pinref part="C27" gate="G$1" pin="+"/>
+<wire x1="144.78" y1="33.02" x2="149.86" y2="33.02" width="0.1524" layer="91"/>
+<wire x1="149.86" y1="33.02" x2="154.94" y2="33.02" width="0.1524" layer="91"/>
+<junction x="154.94" y="33.02"/>
+<pinref part="C28" gate="G$1" pin="1"/>
+<junction x="144.78" y="33.02"/>
+<pinref part="C5" gate="G$1" pin="1"/>
+<junction x="149.86" y="33.02"/>
+<wire x1="154.94" y1="33.02" x2="167.64" y2="33.02" width="0.1524" layer="91"/>
+<wire x1="167.64" y1="33.02" x2="167.64" y2="38.1" width="0.1524" layer="91"/>
+<pinref part="F1" gate="F1" pin="1"/>
+</segment>
+</net>
