File: hardware/sch-pcb files/BLL-EBOOK-3506.brd (EAGLE design)
At the start: 99.2 x 61.7 mm, 57 parts, among them IC1 RT9080-33GJ5, J1 541323462, J2 MSD-3-A, J3 DX07S016JA1R1500, J4 BATT PAD, Q1 IRLML6402TRPBF, U2 TPS65185RGZR, U3 USBLC6-2P6

Commit message: new core design for bll pilot
Parts:
- added U$3: LUCKFOX_CORE3506, Luckfox_Core3506:CORE3506
- U$1: value LUCKFOX_CORE3506 -> IT8951; device Luckfox_Core3506:CORE3506 -> it8951E:LQFP128_STM
- moved U$1 23.5 mm to (47.0, 62.4), turned to 180 degrees
- moved C26 3.30 mm to (26.4, 69.9)
Connections:
- removed net LEH: J1.10
- new net H-CS: U$1.115, U$3.P$17
- new net H-MISO: U$1.118, U$3.P$15
- new net H-MOSI: U$1.117, U$3.P$16
- new net H-SCK: U$1.116, U$3.P$18
- new net N$10: U$1.13
- new net N$22: U$1.14
- new net N$7: U$1.73
- new net N$8: U$1.12
- new net XLE: J1.10, U$1.107
- new net XOE: J1.11, U$1.77
- net 3.3V: now also U$1.1, U$1.126, U$1.20, U$1.33, U$1.45, U$1.60, U$1.75, U$1.94, U$1.99
- net CKV: now also U$1.74
- net D0: now also U$1.82
- net D1: now also U$1.83
- net D2: now also U$1.84
- net D3: now also U$1.85
- net D4: now also U$1.86
- net D5: now also U$1.87
- net D6: now also U$1.88
- net D7: now also U$1.89
- net EP-STV: now also U$1.71
- net GND: now also U$1.104, U$1.113, U$1.120, U$1.125, U$1.128, U$1.21, U$1.37, U$1.61, U$1.76, U$1.97, U$3.P$81, U$3.P$88, U$3.P$89, U$3.P$90; no longer U$1.P$71, U$1.P$81, U$1.P$88, U$1.P$89, U$1.P$90
- net P: now also U$3.P$85, U$3.P$86, U$3.P$87; no longer U$1.P$85, U$1.P$86, U$1.P$87
- net USB+: now also U$3.P$108; no longer U$1.P$108
- net USB-: now also U$3.P$109; no longer U$1.P$109
- net XCL: now also U$1.109
- net XSTL: now also U$1.108
Routing:
- net GND: track 377.7 -> 511.8 mm, vias 9 -> 16
- net LEH: track 37.3 -> 0.00 mm, vias 2 -> 0
- net XLE: track 0.00 -> 31.8 mm, vias 0 -> 2
- net D0: track 37.8 -> 17.3 mm
- net D1: track 36.6 -> 17.3 mm
- net D2: track 35.5 -> 17.3 mm
- net XOE: track 0.00 -> 18.0 mm
- net D6: track 34.3 -> 17.1 mm
- net D3: track 34.4 -> 17.2 mm
- net D7: track 33.7 -> 17.0 mm
- net D4: track 33.3 -> 17.2 mm
- net D5: track 32.1 -> 17.1 mm
- net SCK: track 17.5 -> 3.77 mm
- net EP-VCOM: track 64.9 -> 77.4 mm
- net 3.3V: track 159.8 -> 171.2 mm, vias 5 -> 4
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Other:
- board size 99.2 x 61.7 mm -> 99.2 x 73.2 mm

Commit message: new schematic update
Parts:
- added U$2: LT8912B, LT8912B:LT8912B
- moved C1 6.12 mm to (18.5, 14.5)
- moved J2 6.12 mm to (7.68, 21.8)
- moved R4 6.12 mm to (20.7, 16.8)
- moved U$3 1.59 mm to (49.8, 32.5), turned to 0 degrees
Connections:
- new net DSI-CKN: U$2.P7, U$3.P$1
- new net DSI-CKP: U$2.P6, U$3.P$2
- new net DSI0-DN: U$2.P1, U$3.P$7
- new net DSI0-DP: U$2.P0, U$3.P$8
- new net DSI1-DN: U$2.P3, U$3.P$4
- new net DSI1-DP: U$2.P2, U$3.P$5
- new net I2C-SCL: U$2.P61, U$3.P$59
- new net I2C-SDA: U$2.P60, U$3.P$58
- net GND: now also U$3.P$3, U$3.P$6, U$3.P$9
Routing:
- net I2C-SDA: track 0.00 -> 59.7 mm, vias 0 -> 2
- net I2C-SCL: track 0.00 -> 59.2 mm, vias 0 -> 2
- net USB+: track 13.2 -> 62.6 mm, vias 0 -> 2
- net USB-: track 13.3 -> 62.0 mm, vias 0 -> 2
- net GND: track 511.8 -> 560.0 mm
- net H-SCK: track 6.05 -> 35.1 mm, vias 0 -> 2
- net H-MOSI: track 5.16 -> 33.8 mm, vias 0 -> 2
- net H-MISO: track 4.98 -> 31.6 mm, vias 0 -> 2
- net H-CS: track 8.92 -> 34.4 mm
- net DSI-CKN: track 0.00 -> 13.7 mm
- net DSI-CKP: track 0.00 -> 13.5 mm
- net DSI1-DN: track 0.00 -> 13.1 mm
- net DSI1-DP: track 0.00 -> 12.9 mm
- net DSI0-DN: track 0.00 -> 12.2 mm
- net DSI0-DP: track 0.00 -> 12.0 mm
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
Commit message: new sch and brd design update
Parts:
- removed R4: 10k, rcl:M0805
- added C29, C30: 22pF, SparkFun-Capacitors:0603
- added C31, C32, C33: 10uF, rcl:C0603
- added C34: 1.0uF, SparkFun-Capacitors:0603
- added FUSE-0603: 500mA, SparkFun-Resistors:0603
- added IC2: RT9080-33GJ5, RT9080-33GJ5:SOT94P280X100-5N
- added IC3: RT9080-18GJ5, RT9080-33GJ5:SOT94P280X100-5N
- added Q2: 27Mhz Osc, crystal-geyer_V1_0:5.0X3.2_2
- added Q3, Q4: AO3400, IRLML6402:SOT23
- added R5, R6: 10k, rcl:M0805
- added U$4: MICROSD-MODULE, micro-sd-module:MICROSD-MOD
- C1: value 100nF -> 10uF
- J2: value MSD-3-A -> HDMR-19-02-F-SM; device MSD-3-A:CUI_MSD-3-A -> HDMR-19-02-F-SM:SAMTEC_HDMR-19-02-F-SM
- moved C1 15.4 mm to (12.4, 28.7), turned to 90 degrees
- moved J2 14.5 mm to (3.56, 35.7)
- moved U$2 4.32 mm to (21.7, 40.8)
Connections:
- removed net CD: C1.1, J2.CD, R4.1
- removed net MISO: J2.7
- removed net MOSI: J2.3
- removed net OUT+: F1.2
- removed net SCK: J2.5
- removed net SCL: R8.1, U2.17
- removed net SDA: R9.1, U2.18
- new net 1.8V: C33.1, IC3.5, U$2.P17, U$2.P34, U$2.P4, U$2.P42, U$2.P56
- new net 3.3V2: C1.1, C32.1, IC2.5, IC3.1, IC3.3, R5.1, R6.1, U$4.P$1
- new net GPIO-HDMI: Q4.1
- new net GPIO-SD: Q3.1
- new net HDMI-CKN: J2.12, U$2.P37
- new net HDMI-CKP: J2.10, U$2.P38
- new net HDMITX0-DN: J2.09, U$2.P40
- new net HDMITX0-DP: J2.07, U$2.P41
- new net HDMITX1-DN: J2.06, U$2.P43
- new net HDMITX1-DP: J2.04, U$2.P44
- new net HDMITX2-DN: J2.03, U$2.P46
- new net HDMITX2-DP: J2.01, U$2.P47
- new net HPD: J2.19, U$2.P13
- new net I2C1-SCL: R8.1, U$3.P$61, U2.17
- new net I2C1-SDA: R9.1, U$3.P$60, U2.18
- new net N$1: C29.2, Q2.1, U$2.P53
- new net N$2: C30.2, Q2.2, U$2.P52
- new net N$30: J2.13
- new net N$31: J2.14
- new net N$32: J2.15
- new net N$33: J2.16
- new net N$35: C34.1, FUSE-0603.1, J2.18
- new net SPI-CLK: U$3.P$21, U$4.P$4
- new net SPI-CS: R5.2, U$3.P$20, U$4.P$2
- new net SPI-MISO: R6.2, U$3.P$22, U$4.P$5
- new net SPI-MOSI: U$3.P$23, U$4.P$3
- new net SW1: Q3.3, U$4.P$6
- new net SW2: C1.2, C29.1, C30.1, C33.2, IC3.2, Q4.3, U$2.P16, U$2.P20, U$2.P26, U$2.P33, U$2.P39, U$2.P45, U$2.P5, U$2.P50, U$2.P55
- net 3.3V: no longer J2.4, R4.2
- net GND: now also C31.2, C32.2, C34.2, IC2.2, J2.02, J2.05, J2.08, J2.11, J2.17, J2.S1, J2.S2, J2.S3, J2.S4, Q3.2, Q4.2, U$3.P$26, U$3.P$47; no longer C1.2, J2.6, J2.G1, J2.G2, J2.G3, J2.G4
- net VIN: now also C31.1, F1.2, FUSE-0603.2, IC2.1, IC2.3
Routing:
- net GND: track 560.0 -> 680.6 mm, vias 16 -> 23
- net VIN: track 107.5 -> 208.0 mm, vias 6 -> 7
- net SW2: track 0.00 -> 86.5 mm, vias 0 -> 9
- net I2C1-SDA: track 0.00 -> 65.8 mm, vias 0 -> 2
- net I2C1-SCL: track 0.00 -> 60.3 mm, vias 0 -> 2
- net 1.8V: track 0.00 -> 56.1 mm, vias 0 -> 6
- net SDA: track 50.3 -> 0.00 mm, vias 1 -> 0
- net SCL: track 49.6 -> 0.00 mm, vias 1 -> 0
- net N$35: track 0.00 -> 47.5 mm, vias 0 -> 2
- net 3.3V2: track 0.00 -> 47.0 mm
- net HPD: track 0.00 -> 28.9 mm
- net SPI-CS: track 0.00 -> 28.7 mm, vias 0 -> 2
- net HDMI-CKP: track 0.00 -> 27.3 mm
- net HDMI-CKN: track 0.00 -> 27.3 mm
- net SPI-CLK: track 0.00 -> 26.6 mm
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
Commit message: updated pcb and schematic design
Parts:
- added C35: 1.0uF, SparkFun-Capacitors:0603
- added C36: 100uF, SparkFun-Capacitors:EIA3528
- added C37: 100nF, SparkFun-Capacitors:0805
- added F2: 1206L150, SparkFun-Fuses:1206
- added Q5: AO3400, IRLML6402:SOT23
- added U$5: USB-WIFI-DONGLE, usb-wifi-dongle:USB-A-SMT-MALE
- moved C28 3.46 mm to (69.7, 45.4)
- moved C27 3.40 mm to (74.7, 45.5)
- moved C5 3.17 mm to (71.9, 45.6)
- moved F1 2.67 mm to (79.1, 46.2)
Connections:
- new net GPIO-USB: Q5.1, U$3.P$97
- new net N$5: F2.2, U$5.VBUS1
- new net P1: C35.1, C36.A, C37.1, F2.1, Q5.2
- new net SPI1-CLK: U$3.P$70
- new net SPI1-CS: U$3.P$64
- new net SPI1-MISO: U$3.P$68
- new net SPI1-MOSI: U$3.P$69
- new net USB1+: U$3.P$110, U$5.D+1
- new net USB1-: U$3.P$111, U$5.D-1
- net GND: now also C35.2, C36.C, C37.2, U$3.P$100, U$3.P$107, U$3.P$118, U$3.P$19, U$3.P$71, U$5.GND1
- net GPIO-HDMI: now also U$3.P$28
- net GPIO-SD: now also U$3.P$30
- net VIN: now also Q5.3
Routing:
- net GND: track 680.6 -> 731.8 mm, vias 23 -> 21
- net USB1-: track 0.00 -> 34.0 mm
- net USB1+: track 0.00 -> 30.6 mm
- net P1: track 0.00 -> 17.5 mm
- net GPIO-HDMI: track 0.00 -> 16.7 mm, vias 0 -> 2
- net VBUS: track 50.5 -> 38.7 mm
- net VIN: track 208.0 -> 219.5 mm
- net GPIO-USB: track 0.00 -> 11.3 mm
- net GPIO-SD: track 0.00 -> 5.67 mm
- net N$5: track 0.00 -> 4.25 mm
- net H-MISO: track 31.6 -> 34.2 mm
- net H-SCK: track 35.1 -> 37.6 mm
- net H-CS: track 34.4 -> 36.7 mm
- net H-MOSI: track 33.8 -> 35.8 mm
- net P: track 17.4 -> 16.7 mm
Other:
- board text added: "charge module output 5v"
- board text removed: "IN FROM BAT"
- board text removed: "to charge module"

Commit message: updated pcb and schematic files.
Parts:
- added J5: (no value), SparkFun-Connectors:1X02_LOCK
- added R4, R7: 33, SparkFun-Resistors:0603
- renumbered U$2 to LT8912
Connections:
- new net I2C0-SCL: U$3.P$63
- new net I2C0-SDA: U$3.P$62
- new net N$6: J5.1, R4.2
- new net N$9: J5.2, R7.2
- new net UART0-RX: R7.1, U$3.P$56
- new net UART0-TX: R4.1, U$3.P$57
Routing:
- net VIN: track 219.5 -> 226.2 mm
- net GND: track 731.8 -> 737.5 mm
- net N$9: track 0.00 -> 3.52 mm
- net N$6: track 0.00 -> 3.37 mm
- net UART0-TX: track 0.00 -> 3.08 mm
- net UART0-RX: track 0.00 -> 2.93 mm
- net I2C1-SDA: track 65.8 -> 66.9 mm
- net EPD-VDD: track 68.5 -> 67.7 mm
- net USB+: track 62.6 -> 61.8 mm
- net I2C1-SCL: track 60.5 -> 61.3 mm
- net P37: track 18.2 -> 18.7 mm
Other:
- board text added: "RX-TX"
- board text added: "UART"
