File: hardware/sch-pcb files/BLL-EBOOK-3506.sch (EAGLE design)
At the start: 57 parts, among them IC1 RT9080-33GJ5, J1 541323462, J2 MSD-3-A, J3 DX07S016JA1R1500, J4 BATT PAD, Q1 IRLML6402TRPBF, U2 TPS65185RGZR, U3 USBLC6-2P6

Commit message: new core design for bll pilot
Parts:
- added U$3: LUCKFOX_CORE3506, Luckfox_Core3506:LUCKFOX_CORE3506
- U$1: value LUCKFOX_CORE3506 -> IT8951; device Luckfox_Core3506:LUCKFOX_CORE3506 -> it8951E:IT8951
Connections:
- removed net LEH: J1.10
- new net H-CS: U$1.SPI-CS-N, U$3.SPI2-CSN
- new net H-MISO: U$1.SPI-SO, U$3.SPI2-MISO
- new net H-MOSI: U$1.SPI-SI, U$3.SPI2-MOSI
- new net H-SCK: U$1.SPI-SCK, U$3.SPI2-CLK
- new net N$10: U$1.HOST-HRDY
- new net N$22: U$1.HOST-HIRQ
- new net N$7: U$1.GD-RL
- new net N$8: U$1.HOST-DC
- new net XLE: J1.10, U$1.SDLE
- new net XOE: J1.11, U$1.SDOE
- net 3.3V: now also U$1.VCC33A, U$1.VCC3IO, U$1.VCC3IO-2, U$1.VCC3IO1, U$1.VCC3IO3, U$1.VCCK, U$1.VCCK2, U$1.VCCK3, U$1.VS33D
- net CKV: now also U$1.GD-CLK
- net D0: now also U$1.SDDO0
- net D1: now also U$1.SDDO1
- net D2: now also U$1.SDDO2
- net D3: now also U$1.SDDO3
- net D4: now also U$1.SDDO4
- net D5: now also U$1.SDDO5
- net D6: now also U$1.SDDO6
- net D7: now also U$1.SDDO7
- net EP-STV: now also U$1.GD-SPV
- net GND: now also U$1.GND-A, U$1.GND1, U$1.GND2, U$1.GND3, U$1.GND4, U$1.GND6, U$3.GND10, U$3.GND11, U$3.GND8, U$3.GND9; no longer U$1.GND11
- net P: now also U$3.VCC-5V1, U$3.VCC-5V2, U$3.VCC-5V3; no longer U$1.VCC-5V1, U$1.VCC-5V2, U$1.VCC-5V3
- net USB+: now also U$3.USB0-DP; no longer U$1.USB0-DP
- net USB-: now also U$3.USB0-DN; no longer U$1.USB0-DN
- net XCL: now also U$1.SDCLK
- net XSTL: now also U$1.SDSHR
Other:
- note added: "BLL Ebook Reader Based on Luckfox Core 3506B EPDC IT8951E-64"
- note removed: "BLL Ebook Reader Based on Luckfox Core3506"

Commit message: new schematic update
Parts:
- added U$2: LT8912B, LT8912B:LT8912B
Connections:
- new net DSI-CKN: U$2.MIPI-RX-CKN, U$3.DSI-CLKN
- new net DSI-CKP: U$2.MIPI-RX-CKP, U$3.DSI-CLKP
- new net DSI0-DN: U$2.MIPI-RX0-DN, U$3.DSI-D0N
- new net DSI0-DP: U$2.MIPI-RX0-DP, U$3.DSI-D0P
- new net DSI1-DN: U$2.MIPI-RX1-DN, U$3.DSI-D1N
- new net DSI1-DP: U$2.MIPI-RX1-DP, U$3.DSI-D1P
- new net I2C-SCL: U$2.S-SCL, U$3.I2C2-SCL
- new net I2C-SDA: U$2.S-SDA, U$3.I2C2-SDA
- net GND: now also U$3.GND, U$3.GND2, U$3.GND3
Other:
- note added: "DSI-2-HDMI/LVDS-out"
- note added: "ePaper Display Controller"
Changed lines of the file:
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@@
 <part name="SUPPLY17" library="supply2" library_urn="urn:adsk.eagle:library:372" deviceset="GND" device=""/>
 <part name="SUPPLY18" library="supply2" library_urn="urn:adsk.eagle:library:372" deviceset="GND" device=""/>
+<part name="U$2" library="LT8912B" deviceset="LT8912B" device=""/>
+<part name="SUPPLY19" library="supply2" library_urn="urn:adsk.eagle:library:372" deviceset="GND" device=""/>
 </parts>
 <sheets>
@@
 <plain>
 <text x="-200.66" y="78.74" size="5.08" layer="91">CONEXION USB C</text>
-<text x="-86.36" y="83.82" size="4.5" layer="91">PUERTO MICRO SD</text>
-<text x="-220.98" y="27.94" size="4.5" layer="91">PWR 3.3V</text>
-<text x="-144.78" y="22.86" size="4.5" layer="91">battery/usb
+<text x="-88.9" y="88.9" size="4.5" layer="91">PUERTO MICRO SD</text>
+<text x="-205.74" y="27.94" size="4.5" layer="91">PWR 3.3V</text>
+<text x="-139.7" y="27.94" size="4.5" layer="91">battery/usb
 switching</text>
-<text x="-226.06" y="-20.32" size="4.5" layer="91">ePaper Display Power</text>
+<text x="-170.18" y="-15.24" size="4.5" layer="91">ePaper Display Power</text>
 <text x="193.04" y="63.5" size="4.5" layer="91">ePaper Display Connector
 34pin 0.5 mm pitch</text>
@@
 Based on Luckfox Core 3506B
 EPDC IT8951E-64</text>
+<text x="347.98" y="121.92" size="4.5" layer="91">ePaper Display Controller
+</text>
+<text x="50.8" y="-86.36" size="5.08" layer="91">DSI-2-HDMI/LVDS-out</text>
 </plain>
 <instances>
@@
 <instance part="SUPPLY18" gate="GND" x="421.64" y="81.28" smashed="yes">
 <attribute name="VALUE" x="419.735" y="78.105" size="1.778" layer="96"/>
+</instance>
+<instance part="U$2" gate="G$1" x="78.74" y="-142.24" smashed="yes"/>
+<instance part="SUPPLY19" gate="GND" x="2.54" y="43.18" smashed="yes">
+<attribute name="VALUE" x="0.635" y="40.005" size="1.778" layer="96"/>
 </instance>
 </instances>
@@
 <junction x="132.08" y="48.26"/>
 </segment>
+<segment>
+<pinref part="U$3" gate="G$1" pin="GND"/>
+<pinref part="SUPPLY19" gate="GND" pin="GND"/>
+<wire x1="27.94" y1="45.72" x2="7.62" y2="45.72" width="0.1524" layer="91"/>
+<pinref part="U$3" gate="G$1" pin="GND2"/>
+<wire x1="27.94" y1="38.1" x2="7.62" y2="38.1" width="0.1524" layer="91"/>
+<wire x1="7.62" y1="38.1" x2="7.62" y2="45.72" width="0.1524" layer="91"/>
+<wire x1="7.62" y1="45.72" x2="2.54" y2="45.72" width="0.1524" layer="91"/>
+<pinref part="U$3" gate="G$1" pin="GND3"/>
+<wire x1="27.94" y1="30.48" x2="7.62" y2="30.48" width="0.1524" layer="91"/>
+<wire x1="7.62" y1="30.48" x2="7.62" y2="38.1" width="0.1524" layer="91"/>
+<junction x="7.62" y="38.1"/>
+</segment>
 </net>
 <net name="VBUS" class="0">
@@
 <pinref part="U$1" gate="G$1" pin="HOST-HIRQ"/>
 <wire x1="327.66" y1="22.86" x2="314.96" y2="22.86" width="0.1524" layer="91"/>
+</segment>
+</net>
+<net name="DSI-CKN" class="0">
+<segment>
+<pinref part="U$3" gate="G$1" pin="DSI-CLKN"/>
+<wire x1="27.94" y1="50.8" x2="12.7" y2="50.8" width="0.1524" layer="91"/>
+<label x="12.7" y="50.8" size="1.778" layer="95"/>
+</segment>
+<segment>
+<pinref part="U$2" gate="G$1" pin="MIPI-RX-CKN"/>
+<wire x1="43.18" y1="-142.24" x2="30.48" y2="-142.24" width="0.1524" layer="91"/>
+<label x="30.48" y="-142.24" size="1.778" layer="95"/>
+</segment>
+</net>
+<net name="DSI-CKP" class="0">
+<segment>
+<pinref part="U$3" gate="G$1" pin="DSI-CLKP"/>
+<wire x1="27.94" y1="48.26" x2="12.7" y2="48.26" width="0.1524" layer="91"/>
+<label x="12.7" y="48.26" size="1.778" layer="95"/>
+</segment>
+<segment>
+<pinref part="U$2" gate="G$1" pin="MIPI-RX-CKP"/>
+<wire x1="43.18" y1="-139.7" x2="30.48" y2="-139.7" width="0.1524" layer="91"/>
+<label x="30.48" y="-139.7" size="1.778" layer="95"/>
+</segment>
+</net>
+<net name="DSI1-DN" class="0">
+<segment>
+<pinref part="U$3" gate="G$1" pin="DSI-D1N"/>
+<wire x1="27.94" y1="43.18" x2="12.7" y2="43.18" width="0.1524" layer="91"/>
+<label x="12.7" y="43.18" size="1.778" layer="95"/>
+</segment>
+<segment>
+<pinref part="U$2" gate="G$1" pin="MIPI-RX1-DN"/>
+<wire x1="43.18" y1="-132.08" x2="30.48" y2="-132.08" width="0.1524" layer="91"/>
+<label x="30.48" y="-132.08" size="1.778" layer="95"/>
+</segment>
+</net>
+<net name="DSI1-DP" class="0">
+<segment>
+<pinref part="U$3" gate="G$1" pin="DSI-D1P"/>
+<wire x1="27.94" y1="40.64" x2="12.7" y2="40.64" width="0.1524" layer="91"/>
+<label x="12.7" y="40.64" size="1.778" layer="95"/>
+</segment>
+<segment>
+<pinref part="U$2" gate="G$1" pin="MIPI-RX1-DP"/>
+<wire x1="43.18" y1="-129.54" x2="30.48" y2="-129.54" width="0.1524" layer="91"/>
+<label x="30.48" y="-129.54" size="1.778" layer="95"/>
+</segment>
+</net>
+<net name="DSI0-DN" class="0">
+<segment>
+<pinref part="U$3" gate="G$1" pin="DSI-D0N"/>
+<wire x1="27.94" y1="35.56" x2="12.7" y2="35.56" width="0.1524" layer="91"/>
+<label x="12.7" y="35.56" size="1.778" layer="95"/>
+</segment>
+<segment>
+<pinref part="U$2" gate="G$1" pin="MIPI-RX0-DN"/>
+<wire x1="43.18" y1="-127" x2="30.48" y2="-127" width="0.1524" layer="91"/>
+<label x="30.48" y="-127" size="1.778" layer="95"/>
+</segment>
+</net>
+<net name="DSI0-DP" class="0">
+<segment>
+<pinref part="U$3" gate="G$1" pin="DSI-D0P"/>
+<wire x1="27.94" y1="33.02" x2="12.7" y2="33.02" width="0.1524" layer="91"/>
+<label x="12.7" y="33.02" size="1.778" layer="95"/>
+</segment>
+<segment>
+<pinref part="U$2" gate="G$1" pin="MIPI-RX0-DP"/>
+<wire x1="43.18" y1="-124.46" x2="30.48" y2="-124.46" width="0.1524" layer="91"/>
+<label x="30.48" y="-124.46" size="1.778" layer="95"/>
+</segment>
+</net>
+<net name="I2C-SDA" class="0">
+<segment>
+<pinref part="U$3" gate="G$1" pin="I2C2-SDA"/>
+<wire x1="111.76" y1="-38.1" x2="111.76" y2="-48.26" width="0.1524" layer="91"/>
+<label x="111.76" y="-50.8" size="1.778" layer="95" rot="R90"/>
+</segment>
+<segment>
+<pinref part="U$2" gate="G$1" pin="S-SDA"/>
+<wire x1="71.12" y1="-106.68" x2="71.12" y2="-96.52" width="0.1524" layer="91"/>
+<label x="71.12" y="-104.14" size="1.778" layer="95" rot="R90"/>
+</segment>
+</net>
+<net name="I2C-SCL" class="0">
+<segment>
+<pinref part="U$3" gate="G$1" pin="I2C2-SCL"/>
+<wire x1="114.3" y1="-38.1" x2="114.3" y2="-48.26" width="0.1524" layer="91"/>
+<label x="114.3" y="-50.8" size="1.778" layer="95" rot="R90"/>
+</segment>
+<segment>
+<pinref part="U$2" gate="G$1" pin="S-SCL"/>
+<wire x1="68.58" y1="-106.68" x2="68.58" y2="-99.06" width="0.1524" layer="91"/>
+<wire x1="68.58" y1="-96.52" x2="68.58" y2="-99.06" width="0.1524" layer="91"/>
+<label x="68.58" y="-104.14" size="1.778" layer="95" rot="R90"/>
 </segment>
 </net>
@@
 for full support of labels.
 </note>
+<note version="8.5" severity="warning">
+Since Version 8.5, EAGLE supports locking for holes, vias, wires and polygons.
+The locking property on all objects of these types will not be understood in this version.
+</note>
 </compatibility>

Commit message: new sch and brd design update
Parts:
- removed R4: 10k, rcl:R-US_M0805
- added C29, C30: 22pF, SparkFun-Capacitors:22PF-0603-50V-5%
- added C31, C32, C33: 10uF, rcl:C-USC0603
- added C34: 1.0uF, SparkFun-Capacitors:1.0UF-0603-16V-10%
- added FUSE-0603: 500mA, SparkFun-Resistors:1.8MOHM
- added IC2: RT9080-33GJ5, RT9080-33GJ5:RT9080-33GJ5
- added IC3: RT9080-18GJ5, RT9080-33GJ5:RT9080-33GJ5
- added Q2: 27Mhz Osc, crystal-geyer_V1_0:KX-9B
- added Q3, Q4: AO3400, IRLML6402:IRLML6402TRPBF
- added R5, R6: 10k, rcl:R-US_M0805
- added U$4: MICROSD-MODULE, micro-sd-module:MICROSD-MODULE
- C1: value 100nF -> 10uF
- J2: value MSD-3-A -> HDMR-19-02-F-SM; device MSD-3-A:MSD-3-A -> HDMR-19-02-F-SM:HDMR-19-02-F-SM
Connections:
- removed net CD: C1.1, J2.CD, R4.1
- removed net MISO: J2.DAT0
- removed net MOSI: J2.CMD
- removed net OUT+: F1.2
- removed net SCK: J2.CLK
- removed net SCL: R8.1, U2.SCL
- removed net SDA: R9.1, U2.SDA
- new net 1.8V: C33.1, IC3.VOUT, U$2.VCCA-HDMITX, U$2.VCCA-MIPI-RX, U$2.VDD, U$2.VDD2, U$2.VDD3
- new net 3.3V2: C1.1, C32.1, IC2.VOUT, IC3.EN, IC3.VIN, R5.1, R6.1, U$4.3V3
- new net GPIO-HDMI: Q4.G
- new net GPIO-SD: Q3.G
- new net HDMI-CKN: J2.12, U$2.HDMITX-CKN
- new net HDMI-CKP: J2.10, U$2.HDMITX-CKP
- new net HDMITX0-DN: J2.09, U$2.HDMITX0-DN
- new net HDMITX0-DP: J2.07, U$2.HDMITX0-DP
- new net HDMITX1-DN: J2.06, U$2.HDMITX1-DN
- new net HDMITX1-DP: J2.04, U$2.HDMITX1-DP
- new net HDMITX2-DN: J2.03, U$2.HDMITX2-DN
- new net HDMITX2-DP: J2.01, U$2.HDMITX2-DP
- new net HPD: J2.19, U$2.HPD-CBUS
- new net I2C1-SCL: R8.1, U$3.SPI0-MOSI, U2.SCL
- new net I2C1-SDA: R9.1, U$3.SPI0-MISO, U2.SDA
- new net N$1: C29.2, Q2.1, U$2.XTAL0
- new net N$2: C30.2, Q2.2, U$2.XTALI
- new net N$30: J2.13
- new net N$31: J2.14
- new net N$32: J2.15
- new net N$33: J2.16
- new net N$35: C34.1, FUSE-0603.1, J2.18
- new net SPI-CLK: U$3.FSPI-CLK, U$4.CLK
- new net SPI-CS: R5.2, U$3.FSPI-CSN, U$4.CS
- new net SPI-MISO: R6.2, U$3.FSPI-D0, U$4.MISO
- new net SPI-MOSI: U$3.FSPI-D1, U$4.MOSI
- new net SW1: Q3.D, U$4.GND
- new net SW2: C1.2, C29.1, C30.1, C33.2, IC3.GND, Q4.D, U$2.VSS, U$2.VSS2, U$2.VSS3, U$2.VSSA-HDMIPLL, U$2.VSSA-HDMITX, U$2.VSSA-HDMITX2, U$2.VSSA-LVDSPLL, U$2.VSSA-LVDSTX, U$2.VSSA-MIPI-RX
- net 3.3V: no longer J2.VDD, R4.2
- net GND: now also C31.2, C32.2, C34.2, IC2.GND, J2.02, J2.05, J2.08, J2.11, J2.17, J2.SHIELD, Q3.S, Q4.S, U$3.GND5, U$3.GND6; no longer C1.2, J2.COVER_GND, J2.VSS
- net I2C-SCL: now also U$3.SPI0-CSN0; no longer U$3.I2C2-SCL
- net I2C-SDA: now also U$3.P$58; no longer U$3.I2C2-SDA
- net VIN: now also C31.1, F1.2, FUSE-0603.2, IC2.EN, IC2.VIN
Other:
- note added: "1.8V PWR LT8912B"
- note added: "HDMI Out"
- note added: "MICRO SD MODULE"
- note added: "PWR SWITCH HDMI-SD MOSFETS-N AO3400"
- note removed: "PUERTO MICRO SD"
- moved on the sheet: C1, C26, F1, IC1

Commit message: updated pcb and schematic design
Parts:
- added C35: 1.0uF, SparkFun-Capacitors:1.0UF-0603-16V-10%-X7R
- added C36: 100uF, SparkFun-Capacitors:100UF-POLAR-EIA3528-10V-20%(TANT)
- added C37: 100nF, SparkFun-Capacitors:CAP-0805
- added F2: 1206L150, SparkFun-Fuses:PPTC_6V500MA-2
- added Q5: AO3400, IRLML6402:IRLML6402TRPBF
- added U$5: USB-WIFI-DONGLE, usb-wifi-dongle:USB-WIFI-DONGLE
Connections:
- new net GPIO-USB: Q5.G, U$3.P$97
- new net N$5: F2.2, U$5.P$4
- new net P1: C35.1, C36.+, C37.1, F2.1, Q5.S
- new net SPI1-CLK: U$3.SPI1-CLK
- new net SPI1-CS: U$3.SPI1-CSN0
- new net SPI1-MISO: U$3.SPI1-MISO
- new net SPI1-MOSI: U$3.SPI1-MOSI
- new net USB1+: U$3.USB1-DP, U$5.P$2
- new net USB1-: U$3.USB1-DN, U$5.P$3
- net GND: now also C35.2, C36.-, C37.2, U$3.GND12, U$3.GND13, U$3.GND14, U$3.GND4, U$3.GND7, U$5.P$1
- net GPIO-HDMI: now also U$3.P$28
- net GPIO-SD: now also U$3.P$30
- net VIN: now also Q5.D
Other:
- note added: "USB Dongle Port"

Commit message: updated pcb and schematic files.
Parts:
- added J5: (no value), SparkFun-Connectors:CONN_02LOCK
- added R4, R7: 33, SparkFun-Resistors:33OHM-0603-1/10W-1%
- renumbered U$2 to LT8912
Connections:
- new net I2C0-SCL: U$3.SPI0-CSN1
- new net I2C0-SDA: U$3.SPI0-CLK
- new net N$6: J5.1, R4.2
- new net N$9: J5.2, R7.2
- new net UART0-RX: R7.1, U$3.UART0-RX
- new net UART0-TX: R4.1, U$3.UART0-TX
Other:
- note added: "UART0-Debug Port"
